File: nixie-ps.sch (KiCad schematic (older format))
At the start: 17 parts, among them J1 Conn_01x04_Male, J2 Conn_01x04_Male, Q1 IRFH5106PBF, T1 EFD15_2WI, U1 LM3488MM

Commit message: Replace IRFH5106PBF to RFH7185TRPBF Replace resistor Isense footprint to bigger one Also update ltspice scheme with last changes
Parts:
- removed Q1: IRFH5106PBF, lib_fp:PQFN_5X6MM, symbol esynr3z_TransistorFET:IRFH5106PBF
- added Q1: IRFH7185TRPBF, lib_fp:PQFN_5X6MM, symbol esynr3z_TransistorFET:IRFH7185TRPBF
- R5: value 0.01 -> 0.02; footprint lib_fp:0805 -> lib_fp:2010
Changed lines of the file:
@@
-$EndComp
-$Comp
-L esynr3z_TransistorFET:IRFH5106PBF Q1
-U 1 1 5B2E3CFA
-P 5850 3100
-F 0 "Q1" H 5958 3153 60  0000 L CNN
-F 1 "IRFH5106PBF" H 5200 3300 60  0000 L CNN
-F 2 "lib_fp:PQFN_5X6MM" H 6050 3300 60  0001 L CNN
-F 3 "https://www.infineon.com/dgdl/irfh5106pbf.pdf?fileId=5546d462533600a40153561ae5e81ea6" H 6050 3400 60  0001 L CNN
-F 4 "HEXFET MOSFET N-channel 60V 100A 5.6mOhm PQFN 5x6" H 6050 3500 60  0001 L CNN "Description"
-F 5 "Infineon Technologies" H 6050 3600 60  0001 L CNN "Manufacturer"
-	1    5850 3100
-	1    0    0    -1
 $EndComp
 $Comp
@@
 P 5850 3850
 F 0 "R5" H 5920 3896 50  0000 L CNN
-F 1 "0.01" H 5920 3805 50  0000 L CNN
-F 2 "lib_fp:0805" V 5780 3850 50  0001 C CNN
+F 1 "0.02" H 5920 3805 50  0000 L CNN
+F 2 "lib_fp:2010" V 5780 3850 50  0001 C CNN
 F 3 "~" H 5850 3850 50  0001 C CNN
 	1    5850 3850
@@
 Wire Wire Line
 	7950 2550 7950 2800
+$Comp
+L esynr3z_TransistorFET:IRFH7185TRPBF Q1
+U 1 1 5B3A8C4D
+P 5850 3100
+F 0 "Q1" H 5958 3153 60  0000 L CNN
+F 1 "IRFH7185TRPBF" H 5050 3350 60  0000 L CNN
+F 2 "lib_fp:PQFN_5X6MM" H 6050 3300 60  0001 L CNN
+F 3 "https://www.infineon.com/dgdl/irfh7185pbf.pdf?fileId=5546d462533600a40153561ee0b11ee1" H 6050 3400 60  0001 L CNN
+F 4 "HEXFET MOSFET N-channel 100V 123A 5.2mOhm PQFN 5x6" H 6050 3500 60  0001 L CNN "Description"
+F 5 "Infineon Technologies" H 6050 3600 60  0001 L CNN "Manufacturer"
+	1    5850 3100
+	1    0    0    -1
+$EndComp
 $EndSCHEMATC

Commit message: Make project fully portable
Parts:
- C1: symbol Device:CP1 -> nixie-ps:Device_CP1
- C2, C3, C4: symbol Device:C -> nixie-ps:Device_C
- D1: symbol esynr3z_DiodeRectifier:E1G -> nixie-ps:esynr3z_DiodeRectifier_E1G
- D2: symbol esynr3z_DiodeTVS:SMBJ30CA -> nixie-ps:esynr3z_DiodeTVS_SMBJ30CA
- J1, J2: symbol Connector:Conn_01x04_Male -> nixie-ps:Connector_Conn_01x04_Male
- Q1: symbol esynr3z_TransistorFET:IRFH7185TRPBF -> nixie-ps:esynr3z_TransistorFET_IRFH7185TRPBF
- R1, R2, R3, R4, R5: symbol Device:R -> nixie-ps:Device_R
- RV1: symbol esynr3z_Potentiometer:PVZ3A -> nixie-ps:esynr3z_Potentiometer_PVZ3A
- T1: symbol esynr3z_Transformer:EFD15_2WI -> nixie-ps:esynr3z_Transformer_EFD15_2WI
- U1: symbol esynr3z_RegulatorSwitching:LM3488MM -> nixie-ps:esynr3z_RegulatorSwitching_LM3488MM
Changed lines of the file:
@@
 $EndDescr
 $Comp
-L esynr3z_RegulatorSwitching:LM3488MM U1
+L nixie-ps:esynr3z_RegulatorSwitching_LM3488MM U1
 U 1 1 5B2C071A
 P 4850 3200
@@
 $EndComp
 $Comp
-L Device:R R4
+L nixie-ps:Device_R R4
 U 1 1 5B2E29C2
 P 4150 3850
@@
 $EndComp
 $Comp
-L Device:C C4
+L nixie-ps:Device_C C4
 U 1 1 5B2E2B51
 P 6200 3850
@@
 $EndComp
 $Comp
-L Device:CP1 C1
+L nixie-ps:Device_CP1 C1
 U 1 1 5B2E2CE8
 P 4250 2550
@@
 $EndComp
 $Comp
-L esynr3z_DiodeRectifier:E1G D1
+L nixie-ps:esynr3z_DiodeRectifier_E1G D1
 U 1 1 5B2E7F0D
 P 7000 2350
@@
 $EndComp
 $Comp
-L esynr3z_DiodeTVS:SMBJ30CA D2
+L nixie-ps:esynr3z_DiodeTVS_SMBJ30CA D2
 U 1 1 5B2FB57D
 P 6200 3100
@@
 $EndComp
 $Comp
-L esynr3z_Potentiometer:PVZ3A RV1
+L nixie-ps:esynr3z_Potentiometer_PVZ3A RV1
 U 1 1 5B308C77
 P 7650 3800
@@
 $EndComp
 $Comp
-L esynr3z_Transformer:EFD15_2WI T1
+L nixie-ps:esynr3z_Transformer_EFD15_2WI T1
 U 1 1 5B309C28
 P 6350 2550
@@
 $EndComp
 $Comp
-L Device:R R3
+L nixie-ps:Device_R R3
 U 1 1 5B30AA24
 P 3800 3850
@@
 $EndComp
 $Comp
-L Device:C C3
+L nixie-ps:Device_C C3
 U 1 1 5B30AAD8
 P 3800 3500
@@
 $EndComp
 $Comp
-L Device:R R5
+L nixie-ps:Device_R R5
 U 1 1 5B30AF32
 P 5850 3850
@@
 $EndComp
 $Comp
-L Device:R R2
+L nixie-ps:Device_R R2
 U 1 1 5B30AFEC
 P 7650 3450
@@
 $EndComp
 $Comp
-L Device:R R1
+L nixie-ps:Device_R R1
 U 1 1 5B30B03F
 P 7650 2550
@@
 $EndComp
 $Comp
-L Device:C C2
+L nixie-ps:Device_C C2
 U 1 1 5B30B0A5
 P 7250 2550
@@
 	4250 2350 4250 2400
 $Comp
-L power:GND #PWR01
+L nixie-ps:power_GND #PWR01
 U 1 1 5B30B3AF
 P 4000 2800
@@
 $EndComp
 $Comp
-L power:GND #PWR02
+L nixie-ps:power_GND #PWR02
 U 1 1 5B30B404
 P 4250 2800
@@
 $EndComp
 $Comp
-L power:GND #PWR03
+L nixie-ps:power_GND #PWR03
 U 1 1 5B30B4BF
 P 6800 2800
@@
 	7650 3650 7650 3600
 $Comp
-L power:GND #PWR011
+L nixie-ps:power_GND #PWR011
 U 1 1 5B30DC07
 P 7650 4050
@@
 $EndComp
 $Comp
-L power:GND #PWR04
+L nixie-ps:power_GND #PWR04
 U 1 1 5B30E3AA
 P 7250 2800
@@
 $EndComp
 $Comp
-L power:GND #PWR05
+L nixie-ps:power_GND #PWR05
 U 1 1 5B30E76B
 P 7950 2800
@@
 $EndComp
 $Comp
-L power:GND #PWR09
+L nixie-ps:power_GND #PWR09
 U 1 1 5B30EB81
 P 5850 4050
@@
 $EndComp
 $Comp
-L power:GND #PWR08
+L nixie-ps:power_GND #PWR08
 U 1 1 5B30EF42
 P 5250 4050
@@
 $EndComp
 $Comp
-L power:GND #PWR07
+L nixie-ps:power_GND #PWR07
 U 1 1 5B30F358
 P 4150 4050
@@
 $EndComp
 $Comp
-L power:GND #PWR06
+L nixie-ps:power_GND #PWR06
 U 1 1 5B30F719
 P 3800 4050
@@
 	5850 4000 5850 4050
 $Comp
-L power:GND #PWR010
+L nixie-ps:power_GND #PWR010
 U 1 1 5B361C86
 P 6200 4050
@@
 FA
 $Comp
-L Connector:Conn_01x04_Male J1
+L nixie-ps:Connector_Conn_01x04_Male J1
 U 1 1 5B3899B5
 P 3750 2350
@@
 $EndComp
 $Comp
-L Connector:Conn_01x04_Male J2
+L nixie-ps:Connector_Conn_01x04_Male J2
 U 1 1 5B389BAF
 P 8200 2350
@@
 	7950 2550 7950 2800
 $Comp
-L esynr3z_TransistorFET:IRFH7185TRPBF Q1
+L nixie-ps:esynr3z_TransistorFET_IRFH7185TRPBF Q1
 U 1 1 5B3A8C4D
 P 5850 3100

Commit message: Prepare sch and pcb for generating docs
Parts:
- T1: Sec Sec 160x0.1 -> Sec 200x0.1
Changed lines of the file:
@@
 F 5 "B66414W1008D001" H 6800 3000 50  0001 C CNN "CoilFormer"
 F 6 "Pri 5x0.7" H 6350 2928 50  0000 C CNN "Prim"
-F 7 "Sec 160x0.1" H 6350 2837 50  0000 C CNN "Sec"
+F 7 "Sec 200x0.1" H 6350 2837 50  0000 C CNN "Sec"
 	1    6350 2550
 	1    0    0    -1
