File: nixie-ps.sch (KiCad schematic (older format))
At the start: 17 parts, among them J1 Conn_01x04_Male, J2 Conn_01x04_Male, Q1 IRFH7185TRPBF, T1 EFD15_2WI, U1 LM3488MM

Commit message: Update sch and pcb after latest simulation
Parts:
- removed D2: SMBJ30CA, lib_fp:SMB, symbol nixie-ps:esynr3z_DiodeTVS_SMBJ30CA
- added D2: SMBJ70CA, lib_fp:SMB, symbol nixie-ps:esynr3z_DiodeTVS_SMBJ70CA
- R1: value 470k -> 1.2M
- R2: value 2.2k -> 7.5k
- R5: value 0.02 -> 0.01
- T1: Sec Sec 200x0.1 -> Sec 50x0.2
Changed lines of the file:
@@
 Title "High voltage power supply unit for Nixie tubes"
 Date ""
-Rev "v1.0"
+Rev "v1.1"
 Comp ""
 Comment1 ""
@@
 $EndComp
 $Comp
-L nixie-ps:esynr3z_DiodeTVS_SMBJ30CA D2
-U 1 1 5B2FB57D
-P 6200 3100
-F 0 "D2" V 6147 3203 60  0000 L CNN
-F 1 "SMBJ30CA" V 6253 3203 60  0000 L CNN
-F 2 "lib_fp:SMB" H 6400 3300 60  0001 L CNN
-F 3 "http://www.littelfuse.com/~/media/electronics/datasheets/tvs_diodes/littelfuse_tvs_diode_smbj_datasheet.pdf.pdf" H 6400 3400 60  0001 L CNN
-	1    6200 3100
-	0    1    1    0
-$EndComp
-$Comp
 L nixie-ps:esynr3z_Potentiometer_PVZ3A RV1
 U 1 1 5B308C77
@@
 F 5 "B66414W1008D001" H 6800 3000 50  0001 C CNN "CoilFormer"
 F 6 "Pri 5x0.7" H 6350 2928 50  0000 C CNN "Prim"
-F 7 "Sec 200x0.1" H 6350 2837 50  0000 C CNN "Sec"
+F 7 "Sec 50x0.2" H 6350 2837 50  0000 C CNN "Sec"
 	1    6350 2550
 	1    0    0    -1
@@
 P 5850 3850
 F 0 "R5" H 5920 3896 50  0000 L CNN
-F 1 "0.02" H 5920 3805 50  0000 L CNN
+F 1 "0.01" H 5920 3805 50  0000 L CNN
 F 2 "lib_fp:2010" V 5780 3850 50  0001 C CNN
 F 3 "~" H 5850 3850 50  0001 C CNN
@@
 P 7650 3450
 F 0 "R2" H 7720 3496 50  0000 L CNN
-F 1 "2.2k" H 7720 3405 50  0000 L CNN
+F 1 "7.5k" H 7720 3405 50  0000 L CNN
 F 2 "lib_fp:0805" V 7580 3450 50  0001 C CNN
 F 3 "~" H 7650 3450 50  0001 C CNN
@@
 P 7650 2550
 F 0 "R1" H 7720 2596 50  0000 L CNN
-F 1 "470k" H 7720 2505 50  0000 L CNN
+F 1 "1.2M" H 7720 2505 50  0000 L CNN
 F 2 "lib_fp:0805" V 7580 2550 50  0001 C CNN
 F 3 "~" H 7650 2550 50  0001 C CNN
@@
 	1    0    0    -1
 $EndComp
+$Comp
+L nixie-ps:esynr3z_DiodeTVS_SMBJ70CA D2
+U 1 1 5B829451
+P 6200 3100
+F 0 "D2" V 6147 3203 60  0000 L CNN
+F 1 "SMBJ70CA" V 6253 3203 60  0000 L CNN
+F 2 "lib_fp:SMB" H 6400 3300 60  0001 L CNN
+F 3 "http://www.littelfuse.com/~/media/electronics/datasheets/tvs_diodes/littelfuse_tvs_diode_smbj_datasheet.pdf.pdf" H 6400 3400 60  0001 L CNN
+	1    6200 3100
+	0    1    1    0
+$EndComp
 $EndSCHEMATC

Commit message: Massive update after debuging and testing
Parts:
- R5: value 0.01 -> 0.033
- T1: Prim Pri 5x0.7 -> Pri 10x0.7; Sec Sec 50x0.2 -> Sec 145x0.2
Other:
- note added: "180V 20mA @ 5V in\n180V 40mA @ 12V in"
- note added: "5-12V in"
- note added: "R5 note: this value can be in 0.025 - 0.1 ohm range \ndepending on the desired output current and thermal characteristics"
- note removed: "180 DCV\n25 mA"
- note removed: "5-12 DCV"
- moved on the sheet: C4
Changed lines of the file:
@@
 L nixie-ps:Device_C C4
 U 1 1 5B2E2B51
-P 6200 3850
-F 0 "C4" H 6315 3896 50  0000 L CNN
-F 1 "0.01u" H 6315 3805 50  0000 L CNN
-F 2 "lib_fp:0805" H 6238 3700 50  0001 C CNN
-F 3 "~" H 6200 3850 50  0001 C CNN
-	1    6200 3850
+P 6300 3850
+F 0 "C4" H 6415 3896 50  0000 L CNN
+F 1 "0.01u" H 6415 3805 50  0000 L CNN
+F 2 "lib_fp:0805" H 6338 3700 50  0001 C CNN
+F 3 "~" H 6300 3850 50  0001 C CNN
+	1    6300 3850
 	1    0    0    -1
 $EndComp
@@
 F 4 "B66413U0100K187" H 6800 2900 50  0001 C CNN "Core"
 F 5 "B66414W1008D001" H 6800 3000 50  0001 C CNN "CoilFormer"
-F 6 "Pri 5x0.7" H 6350 2928 50  0000 C CNN "Prim"
-F 7 "Sec 50x0.2" H 6350 2837 50  0000 C CNN "Sec"
+F 6 "Pri 10x0.7" H 6350 2928 50  0000 C CNN "Prim"
+F 7 "Sec 145x0.2" H 6350 2837 50  0000 C CNN "Sec"
 	1    6350 2550
 	1    0    0    -1
@@
 P 5850 3850
 F 0 "R5" H 5920 3896 50  0000 L CNN
-F 1 "0.01" H 5920 3805 50  0000 L CNN
+F 1 "0.033" H 5920 3805 50  0000 L CNN
 F 2 "lib_fp:2010" V 5780 3850 50  0001 C CNN
 F 3 "~" H 5850 3850 50  0001 C CNN
@@
 Wire Wire Line
 	6200 3350 6200 3300
-Wire Wire Line
-	5850 3350 5850 3650
 Connection ~ 5850 3350
 Wire Wire Line
@@
 	7950 2450 7950 2550
 Wire Wire Line
-	6200 4000 6200 4050
+	6300 4000 6300 4050
 Wire Wire Line
 	5250 3700 5250 3750
@@
 	7650 3200 7650 3300
 Wire Wire Line
-	6200 3700 6200 3650
-Wire Wire Line
-	6200 3650 5850 3650
-Connection ~ 5850 3650
-Wire Wire Line
-	5850 3650 5850 3700
+	6300 3700 6300 3650
 Wire Wire Line
 	5850 4000 5850 4050
@@
 L nixie-ps:power_GND #PWR010
 U 1 1 5B361C86
-P 6200 4050
-F 0 "#PWR010" H 6200 3800 50  0001 C CNN
-F 1 "GND" H 6205 3877 50  0000 C CNN
-F 2 "" H 6200 4050 50  0001 C CNN
-F 3 "" H 6200 4050 50  0001 C CNN
-	1    6200 4050
+P 6300 4050
+F 0 "#PWR010" H 6300 3800 50  0001 C CNN
+F 1 "GND" H 6305 3877 50  0000 C CNN
+F 2 "" H 6300 4050 50  0001 C CNN
+F 3 "" H 6300 4050 50  0001 C CNN
+	1    6300 4050
 	1    0    0    -1
 $EndComp
 Text Notes 3300 2450 0    50   ~ 0
-5-12 DCV
+5-12V in
 Text Notes 8400 2350 0    50   ~ 0
-180 DCV\n25 mA
+180V 20mA @ 5V in\n180V 40mA @ 12V in
 Text Label 7650 3200 0    50   ~ 0
 FB
@@
 	0    1    1    0
 $EndComp
+Wire Wire Line
+	5850 3350 5850 3650
+Wire Wire Line
+	5850 3650 6300 3650
+Connection ~ 5850 3650
+Wire Wire Line
+	5850 3650 5850 3700
+Text Notes 5150 4500 0    50   ~ 0
+R5 note: this value can be in 0.025 - 0.1 ohm range \ndepending on the desired output current and thermal characteristics
 $EndSCHEMATC

Commit message: Add BOM
Parts:
- C2: Rating (none) -> 250V X7R
- Q1: Manufacturer Infineon Technologies -> (none)
- RV1: Rating (none) -> 1.5k; Resistance 1.5k -> (none)
- T1: CoilFormer B66414W1008D001 -> (none); Core B66413U0100K187 -> (none); Notes (none) -> Windings: primary 10 turns x 0.7 mm, secondary 145 turns x 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; Prim Pri 10x0.7 -> (none); Sec Sec 145x0.2 -> (none)
- U1: MPN LM3488MM/NOPB -> (none); Manufacturer Texas Instruments -> (none)
Other:
- note added: "Prim 10x0.7\nSec 145x0.2"
Changed lines of the file:
@@
 Title "High voltage power supply unit for Nixie tubes"
 Date ""
-Rev "v1.1"
+Rev "v1.0"
 Comp ""
 Comment1 ""
@@
 F 2 "lib_fp:VSSOP-8_3.0x3.0mm_P0.65mm" H 5050 3400 60  0001 L CNN
 F 3 "http://www.ti.com/lit/ds/symlink/lm3488q-q1.pdf" H 5050 3500 60  0001 L CNN
-F 4 "LM3488MM/NOPB" H 5050 3600 60  0001 L CNN "MPN"
-F 5 "Versatile low-side N-FET high performance controller for switching regulators" H 5050 3700 60  0001 L CNN "Description"
-F 6 "Texas Instruments" H 5050 3800 60  0001 L CNN "Manufacturer"
+F 4 "Versatile low-side N-FET high performance controller for switching regulators" H 5050 3700 60  0001 L CNN "Description"
 	1    4850 3200
 	1    0    0    -1
@@
 F 1 "PVZ3A152" H 7580 3800 50  0000 R CNN
 F 2 "lib_fp:Murata_PVZ3A" H 7800 3850 50  0001 C CNN
-F 3 "" H 7900 3950 50  0001 C CNN
-F 4 "1.5k" H 7580 3709 50  0000 R CNN "Resistance"
+F 3 "~" H 7900 3950 50  0001 C CNN
+F 4 "1.5k" H 7580 3709 50  0000 R CNN "Rating"
 	1    7650 3800
 	1    0    0    -1
@@
 U 1 1 5B309C28
 P 6350 2550
-F 0 "T1" H 6350 3110 50  0000 C CNN
-F 1 "EFD15_2WI" H 6350 3019 50  0000 C CNN
+F 0 "T1" H 6350 2900 50  0000 C CNN
+F 1 "EFD15_2WI" H 6350 2800 50  0000 C CNN
 F 2 "lib_fp:EFD15_B66414W1008D001" H 6350 2550 50  0001 C CNN
-F 3 "~" H 6350 2550 50  0001 C CNN
-F 4 "B66413U0100K187" H 6800 2900 50  0001 C CNN "Core"
-F 5 "B66414W1008D001" H 6800 3000 50  0001 C CNN "CoilFormer"
-F 6 "Pri 10x0.7" H 6350 2928 50  0000 C CNN "Prim"
-F 7 "Sec 145x0.2" H 6350 2837 50  0000 C CNN "Sec"
+F 3 "https://en.tdk.eu/inf/80/db/fer/efd_15_8_5.pdf" H 6350 2550 50  0001 C CNN
+F 4 "Windings: primary 10 turns x 0.7 mm, secondary 145 turns x 0.2 mm; Core: B66413U0100K187; Coil former: B66414W1008D001; Yokes: B66414B2000;" H 6050 3400 50  0001 C CNN "Notes"
 	1    6350 2550
 	1    0    0    -1
@@
 F 2 "lib_fp:1812" H 7288 2400 50  0001 C CNN
 F 3 "~" H 7250 2550 50  0001 C CNN
+F 4 "250V X7R" H 7450 2400 50  0000 C CNN "Rating"
 	1    7250 2550
 	1    0    0    -1
@@
 F 3 "https://www.infineon.com/dgdl/irfh7185pbf.pdf?fileId=5546d462533600a40153561ee0b11ee1" H 6050 3400 60  0001 L CNN
 F 4 "HEXFET MOSFET N-channel 100V 123A 5.2mOhm PQFN 5x6" H 6050 3500 60  0001 L CNN "Description"
-F 5 "Infineon Technologies" H 6050 3600 60  0001 L CNN "Manufacturer"
 	1    5850 3100
 	1    0    0    -1
@@
 Text Notes 5150 4500 0    50   ~ 0
 R5 note: this value can be in 0.025 - 0.1 ohm range \ndepending on the desired output current and thermal characteristics
+Text Notes 6100 2150 0    50   ~ 0
+Prim 10x0.7\nSec 145x0.2
 $EndSCHEMATC
